File: RAMPS-FD/Extra_Mosfets.sch (KiCad schematic (older format))
At the start: 12 parts, among them P901 D12, P902 D2, Q901 DMN2075U, Q902 DMN2075U

Commit message: ramps-FD variant
Parts:
- D13: renamed from D901; footprint (none) -> LEDs:LED_0805; symbol LED -> LED-RESCUE-RAMPS-FD
- D14: renamed from D902; footprint (none) -> LEDs:LED_0805; symbol LED -> LED-RESCUE-RAMPS-FD
- D15: renamed from D903; footprint (none) -> Diodes_SMD:DO-214AB; symbol DIODE -> DIODE-RESCUE-RAMPS-FD
- D16: renamed from D904; footprint (none) -> Diodes_SMD:DO-214AB; symbol DIODE -> DIODE-RESCUE-RAMPS-FD
- P24: renamed from P901; footprint (none) -> Sockets_MOLEX_KK-System:Socket_MOLEX-KK-RM2-54mm_Lock_2pin_straight
- P25: renamed from P902; footprint (none) -> Sockets_MOLEX_KK-System:Socket_MOLEX-KK-RM2-54mm_Lock_2pin_straight
- Q6: renamed from Q901; footprint (none) -> TO_SOT_Packages_SMD:SOT-23_GDS; symbol MOS_N -> MOS_N-RESCUE-RAMPS-FD
- Q7: renamed from Q902; footprint (none) -> TO_SOT_Packages_SMD:SOT-23_GDS; symbol MOS_N -> MOS_N-RESCUE-RAMPS-FD
- R29: renamed from R901; footprint ~ -> Resistors_SMD:R_0805; symbol R -> R-RESCUE-RAMPS-FD
- R30: renamed from R902; footprint ~ -> Resistors_SMD:R_0805; symbol R -> R-RESCUE-RAMPS-FD
- R31: renamed from R905; footprint (none) -> Resistors_SMD:R_0805; symbol R -> R-RESCUE-RAMPS-FD
- R32: renamed from R906; footprint (none) -> Resistors_SMD:R_0805; symbol R -> R-RESCUE-RAMPS-FD
Other:
- moved on the sheet: P24, P25
