File: RAMPS-FD/Power.sch (KiCad schematic (older format))
At the start: 19 parts, among them P101 HB_IN, P103 PS-ON, P105 12V-AUX, P107 MOT_IN, P108 POWER_IN, P219 EXT_5V, U3 LM7812

Commit message: ramps-FD variant
Parts:
- removed JP201: 5V_SEL, ~, symbol JUMP_MINI
- removed P105: 12V-AUX, symbol CONN_2
- removed P219: EXT_5V, symbol CONN_2
- added C1: 22u/35v, Capacitors_SMD:C_0805, symbol C_Small
- added JP2: 5V_SEL, Pin_Headers:Pin_Header_Straight_1x03, symbol JUMP_MINI_3
- added P31: 5v aux, Pin_Headers:Pin_Header_Straight_2x05, symbol conn_2x5
- added P37: aux12_en, Pin_Headers:Pin_Header_Straight_1x02, symbol CONN_01X02
- added P38: aux5_en, Pin_Headers:Pin_Header_Straight_1x02, symbol CONN_01X02
- added P6: 12V aux, Pin_Headers:Pin_Header_Straight_2x05, symbol conn_2x5
- added U1: oki-78sr-5h, TO_SOT_Packages_THT:TO-220_Neutral123_Horizontal_OKI_Mod, symbol 7805
- C2: renamed from C207; footprint (none) -> Capacitors_SMD:C_0805; symbol C -> C-RESCUE-RAMPS-FD
- C3: renamed from C101; footprint (none) -> Capacitors_SMD:c_elec_6.3x7.7; symbol CP1 -> CP1-RESCUE-RAMPS-FD
- C4: renamed from C102; footprint (none) -> Capacitors_SMD:C_0805; symbol C -> C-RESCUE-RAMPS-FD
- D2: renamed from D102; footprint (none) -> TO_SOT_Packages_SMD:TO-277A; symbol DIODE_DUAL_ANODE -> DIODE_DUAL_ANODE-RESCUE-RAMPS-FD
- D3: renamed from D103; footprint (none) -> Diodes_SMD:DO-214AB; symbol DIODE -> DIODE-RESCUE-RAMPS-FD
- F1: renamed from F101; footprint (none) -> RAMPS-FD v3:FUSE-MINI-AUTO
- F2: renamed from F103; footprint (none) -> RAMPS-FD v3:FUSE-MINI-AUTO
- F3: renamed from F102; footprint (none) -> RAMPS-FD v3:FUSE-MINI-AUTO
- JP1: renamed from JP101; footprint (none) -> Pin_Headers:Pin_Header_Straight_1x03
- JP3: renamed from JP102; footprint (none) -> Pin_Headers:Pin_Header_Straight_1x03
- JP4: renamed from JP1; footprint (none) -> Pin_Headers:Pin_Header_Straight_1x02
- P3: renamed from P101; footprint (none) -> RAMPS-FD v3:2p-conn-5,08
- P4: renamed from P107; footprint (none) -> RAMPS-FD v3:2p-conn-5,08
- P5: renamed from P108; footprint (none) -> RAMPS-FD v3:2p-conn-5,08
- P7: renamed from P103; footprint (none) -> Pin_Headers:Pin_Header_Straight_1x01
- U2: renamed from U3; footprint ~ -> TO_SOT_Packages_THT:TO-252-2Lead_edit
Connections:
- net labels added: 5v, AREF
- wire segments 67 -> 107
