File: RAMPS-FD/RAMPS-FD.sch (KiCad schematic (older format))
At the start: 9 parts, among them M101 LOGO_OSHW, M102 PCB_GREEN_RMC, P102 RESET, P106 CONN_3X2, Q101 2N7002, SW101 RESET

Commit message: ramps-FD variant
Parts:
- removed M101: LOGO_OSHW, OSHW_logo_2, symbol LOGO_OSHW
- removed M102: PCB_GREEN_RMC, symbol PCB_GREEN_RMC
- removed P106: CONN_3X2, symbol CONN_3X2
- added LOGO1: OPEN_HARDWARE_1, Symbols:Symbol_OSHW-Logo_SilkScreen, symbol OPEN_HARDWARE_1
- D1: renamed from D101; footprint (none) -> LEDs:LED_0805; symbol LED -> LED-RESCUE-RAMPS-FD
- P2: renamed from P102; footprint (none) -> Pin_Headers:Pin_Header_Straight_1x02
- Q1: renamed from Q101; footprint ~ -> TO_SOT_Packages_SMD:SOT-23_GDS; symbol MOSFET_N -> MOSFET_N-RESCUE-RAMPS-FD
- R1: renamed from R101; footprint (none) -> Resistors_SMD:R_0805; symbol R -> R-RESCUE-RAMPS-FD
- SHIELD1: renamed from SHIELD101; footprint (none) -> arduinodue:ARDUINO_DUE_RAMPS_SHIELD; symbol ARDUINO_DUE_SHIELD -> ARDUINO_DUE_SHIELD-RESCUE-RAMPS-FD
- SW1: renamed from SW101; footprint (none) -> Buttons_Switches_ThroughHole:SW_PUSH_SMALL
Connections:
- net labels removed: A4, A5, A6, A7, AD14, AD15, D32, D39, D43, D45, D47, D50-MISO, D51-MOSI, D52-SCK, UART3_RX_LV, UART3_TX_LV
- wire segments 102 -> 89
- no-connect marks 5 -> 15
Other:
- note added: "SPI Header"
