File: RAMPS-FD/con_inputs.sch (KiCad schematic (older format))
At the start: 7 parts, among them P801 CONN_6, P802 CONN_6X2, U801 4050_RMC

Commit message: ramps-FD variant
Parts:
- removed U801: 4050_RMC, ~, symbol 4050_RMC
- added U11: 4050_RMC, Housings_SSOP:TSSOP-16_4.4x5mm_Pitch0.65mm, symbol 4050_RMC
- C36: renamed from C305; footprint (none) -> Capacitors_SMD:C_0805; symbol C -> C-RESCUE-RAMPS-FD
- JP5: renamed from JP801; footprint ~ -> Pin_Headers:Pin_Header_Straight_1x02
- P22: renamed from P801; footprint (none) -> Pin_Headers:Pin_Header_Straight_1x06
- P23: renamed from P802; footprint (none) -> Pin_Headers:Pin_Header_Straight_2x06
- RP6: renamed from RP801; footprint ~ -> Resistors_SMD:R_Cat16-4
- RP7: renamed from RP802; footprint ~ -> Resistors_SMD:R_Cat16-4
Connections:
- wire segments 61 -> 63
Other:
- moved on the sheet: C36
