File: RAMPS-FD/con_misc.sch (KiCad schematic (older format))
At the start: 17 parts, among them K201 S1, K202 S2, K203 S3, K204 S4, P1 SERIAL1, P2 I2C-1, P211 I2C-0, P213 AUX-4, P214 AUX-2, P215 AUX-3, P216 SERIAL0, U601 24C512

Commit message: ramps-FD variant
Parts:
- removed P213: AUX-4, symbol CONN_18
- removed P214: AUX-2, symbol CONN_5X2
- removed P215: AUX-3, symbol CONN_6X2
- added P16: LCD1, Pin_Headers:Pin_Header_Straight_2x05, symbol conn_2x5
- added P17: LCD2, Pin_Headers:Pin_Header_Straight_2x05, symbol conn_2x5
- added RP5: 10K, Resistors_SMD:R_Cat16-8, symbol R_PACK8
- added U10: 74LVC07A, Housings_SSOP:TSSOP-14_4.4x5mm_Pitch0.65mm, symbol 74LVC07A-RESCUE-RAMPS-FD
- C35: renamed from C601; footprint ~ -> Capacitors_SMD:C_0805; symbol C -> C-RESCUE-RAMPS-FD
- K1: renamed from K201; footprint (none) -> Pin_Headers:Pin_Header_Straight_1x03
- K2: renamed from K202; footprint (none) -> Pin_Headers:Pin_Header_Straight_1x03
- K3: renamed from K203; footprint (none) -> Pin_Headers:Pin_Header_Straight_1x03
- K4: renamed from K204; footprint (none) -> Pin_Headers:Pin_Header_Straight_1x03
- P12: renamed from P216; footprint (none) -> Pin_Headers:Pin_Header_Straight_1x06
- P13: renamed from P1; footprint (none) -> Pin_Headers:Pin_Header_Straight_1x06
- P14: renamed from P211; footprint (none) -> Pin_Headers:Pin_Header_Straight_1x04
- P15: renamed from P2; footprint (none) -> Pin_Headers:Pin_Header_Straight_1x04
- R17: renamed from R211; footprint (none) -> Resistors_SMD:R_0805; symbol R -> R-RESCUE-RAMPS-FD
- R18: renamed from R1; footprint (none) -> Resistors_SMD:R_0805; symbol R -> R-RESCUE-RAMPS-FD
- R19: renamed from R212; footprint (none) -> Resistors_SMD:R_0805; symbol R -> R-RESCUE-RAMPS-FD
- R20: renamed from R2; footprint (none) -> Resistors_SMD:R_0805; symbol R -> R-RESCUE-RAMPS-FD
- U9: renamed from U601; footprint (none) -> Housings_SOIC:SOIC-8-1EP_3.9x4.9mm_Pitch1.27mm
Connections:
- net labels added: GND-II_RevF_Date23Aug2012, LCD_D4, LCD_D5, LCD_D6, LCD_D7, LCD_E, LCD_RS
- net labels removed: A4, A5, A6, A7, AD14, AD15, D32, D39, D43, D45, D47, D50-MISO, D51-MOSI, D52-SCK, UART3_RX_LV, UART3_TX_LV
- wire segments 108 -> 115
- no-connect marks 7 -> 12
Other:
- note added: "LCD"
- note added: "aux4 direct to lcd as well"
- note added: "removed aux 2 for digi pots"
- note added: "routed aux3 direct to LCD header"
- note removed: "Aux2"
- note removed: "Aux3 - SPI"
- note removed: "Aux4 - general IO"
- note removed: "Mega: same signals as \nMISO, MOSI & SCK"
- note removed: "NB This pin is always 5V"
- note removed: "Note: Some addon boards \nconnect this pin to GND."
- note removed: "These are free \nfor LCD panel etc"
- note removed: "These are shared with E1 \nand E2 stepper signals"
