File: RAMPS-FD/con_outputs.sch (KiCad schematic (older format))
At the start: 24 parts, among them P218 D11, P403 D9, P404 D8, P405 D10, Q201 IRLB8743PBF, Q202 IRLB8743PBF, Q203 IRLB8743PBF, Q206 IRLB8743PBF

Commit message: ramps-FD variant
Parts:
- D10: renamed from D202; footprint (none) -> LEDs:LED_0805; symbol LED -> LED-RESCUE-RAMPS-FD
- D11: renamed from D402; footprint (none) -> Diodes_SMD:DO-214AB; symbol DIODE -> DIODE-RESCUE-RAMPS-FD
- D12: renamed from D403; footprint (none) -> Diodes_SMD:DO-214AB; symbol DIODE -> DIODE-RESCUE-RAMPS-FD
- D5: renamed from D201; footprint (none) -> LEDs:LED_0805; symbol LED -> LED-RESCUE-RAMPS-FD
- D6: renamed from D203; footprint (none) -> LEDs:LED_0805; symbol LED -> LED-RESCUE-RAMPS-FD
- D7: renamed from D401; footprint (none) -> Diodes_SMD:DO-214AB; symbol DIODE -> DIODE-RESCUE-RAMPS-FD
- D8: renamed from D404; footprint (none) -> Diodes_SMD:DO-214AB; symbol DIODE -> DIODE-RESCUE-RAMPS-FD
- D9: renamed from D204; footprint (none) -> LEDs:LED_0805; symbol LED -> LED-RESCUE-RAMPS-FD
- P18: renamed from P403; footprint (none) -> RAMPS-FD v3:2p-conn-5,08
- P19: renamed from P404; footprint (none) -> RAMPS-FD v3:2p-conn-5,08
- P20: renamed from P405; footprint (none) -> RAMPS-FD v3:2p-conn-5,08
- P21: renamed from P218; footprint (none) -> RAMPS-FD v3:2p-conn-5,08
- Q2: renamed from Q201; value IRLB8743PBF -> IRFR8314TRPBF; footprint (none) -> TO_SOT_Packages_SMD:TO-252-2Lead_GDS
- Q3: renamed from Q203; value IRLB8743PBF -> IRFR8314TRPBF; footprint (none) -> TO_SOT_Packages_SMD:TO-252-2Lead_GDS
- Q4: renamed from Q206; value IRLB8743PBF -> IRFR8314TRPBF; footprint (none) -> TO_SOT_Packages_SMD:TO-252-2Lead_GDS
- Q5: renamed from Q202; value IRLB8743PBF -> IRFR8314TRPBF; footprint (none) -> TO_SOT_Packages_SMD:TO-252-2Lead_GDS
- R21: renamed from R701; footprint (none) -> Resistors_SMD:R_0805; symbol R -> R-RESCUE-RAMPS-FD
- R22: renamed from R702; footprint (none) -> Resistors_SMD:R_0805; symbol R -> R-RESCUE-RAMPS-FD
- R23: renamed from R219; footprint (none) -> Resistors_SMD:R_0805; symbol R -> R-RESCUE-RAMPS-FD
- R24: renamed from R221; footprint (none) -> Resistors_SMD:R_0805; symbol R -> R-RESCUE-RAMPS-FD
- R25: renamed from R703; footprint (none) -> Resistors_SMD:R_0805; symbol R -> R-RESCUE-RAMPS-FD
- R26: renamed from R704; footprint (none) -> Resistors_SMD:R_0805; symbol R -> R-RESCUE-RAMPS-FD
- R27: renamed from R222; footprint (none) -> Resistors_SMD:R_0805; symbol R -> R-RESCUE-RAMPS-FD
- R28: renamed from R220; footprint (none) -> Resistors_SMD:R_0805; symbol R -> R-RESCUE-RAMPS-FD
Connections:
- net labels added: FET4_G, GND
Other:
- moved on the sheet: P18, P19, P21
