File: RAMPS-FD/e-stop.sch (KiCad schematic (older format))
At the start: 14 parts, among them P302 ESTOP, U1 74ACT125, U2 74ACT244

Commit message: ramps-FD variant
Parts:
- removed R401, R402: 10k, symbol R
- removed RP1, RP2, RP401: 10k, symbol R_PACK4
- removed U1: 74ACT125, symbol 74LS125
- added RP1, RP2: R_PACK8, Resistors_SMD:R_Cat16-8, symbol R_PACK8
- added RP4: R_PACK4, Resistors_SMD:R_Cat16-4, symbol R_PACK4
- added U3: 74ACT244, Housings_SSOP:TSSOP-20_4.4x6.5mm_Pitch0.65mm, symbol 74LS244
- C5: renamed from C1; footprint (none) -> Capacitors_SMD:C_0805; symbol C -> C-RESCUE-RAMPS-FD
- C6: renamed from C2; footprint (none) -> Capacitors_SMD:C_0805; symbol C -> C-RESCUE-RAMPS-FD
- D4: renamed from D301; footprint (none) -> Diodes_SMD:SOD-323; symbol DIODE -> DIODE-RESCUE-RAMPS-FD
- P8: renamed from P302; footprint (none) -> Sockets_MOLEX_KK-System:Socket_MOLEX-KK-RM2-54mm_Lock_2pin_straight
- R2: renamed from R305; footprint (none) -> Resistors_SMD:R_0805; symbol R -> R-RESCUE-RAMPS-FD
- R3: renamed from R304; footprint (none) -> Resistors_SMD:R_0805; symbol R -> R-RESCUE-RAMPS-FD
- RP3: value 10k -> R_PACK4; footprint (none) -> Resistors_SMD:R_Cat16-4
- U4: renamed from U2; footprint (none) -> Housings_SSOP:TSSOP-20_4.4x6.5mm_Pitch0.65mm
Connections:
- wire segments 82 -> 91
- no-connect marks 0 -> 20
