File: RAMPS-FD/steppers.sch (KiCad schematic (older format))
At the start: 15 parts, among them P201 CONN_3X2, P202 CONN_3X2, P203 CONN_3X2, P204 X, P205 Y, P206 Z, U201 X, U202 Y, U203 Z

Commit message: ramps-FD variant
Parts:
- removed C201, C202, C203: 100u 35V, symbol CP1
- removed P201, P202, P203: CONN_3X2, symbol CONN_3X2
- removed R201, R202, R203: 100k, symbol R
- removed U201: X, symbol POLOLU
- removed U202: Y, symbol POLOLU
- removed U203: Z, symbol POLOLU
- added C46, C50, C54, C57, C58, C61, C62, C68, C71: 100n/50v, Capacitors_SMD:C_0805, symbol C
- added C47, C52, C65: 4u7/10v, Capacitors_SMD:C_0805, symbol C
- added C48, C53, C66: 100u/35v, Capacitors_SMD:c_elec_6.3x7.7, symbol CP1_Small
- added C49, C67, C73: 100n50v, Capacitors_SMD:C_0805, symbol C
- added C51, C63, C72: 470n/10v, Capacitors_SMD:C_0805, symbol C
- added C55, C59, C69: 22n/50v, Capacitors_SMD:C_0805, symbol C
- added C56, C60, C70: 1u/50v, Capacitors_SMD:C_0805, symbol C
- added C64: 0.1u, Capacitors_SMD:C_0805, symbol C_Small
- added P30: Z-MOT2, Sockets_MOLEX_KK-System:Socket_MOLEX-KK-RM2-54mm_Lock_4pin_straight, symbol CONN_4
- added P34: Y_SPRD_En, Pin_Headers:Pin_Header_Straight_1x02, symbol CONN_01X02
- added P35: Z_SPRD_En, Pin_Headers:Pin_Header_Straight_1x02, symbol CONN_01X02
- added P36: X_SPRD_En, Pin_Headers:Pin_Header_Straight_1x02, symbol CONN_01X02
- added R44, R45, R50: 2r2, Resistors_SMD:R_0805, symbol R
- added R46, R47, R48, R49, R53, R54: 0r11, Resistors_SMD:R_0805, symbol R
- added R51, R52: 4k7, Resistors_SMD:R_0805, symbol R
- added U13, U14, U16: TMC2130, Housings_DFN_QFN:QFN-36-1EP_5x6mm_Pitch0.5mm, symbol TMC2130-RESCUE-RAMPS-FD
- added U15: DS3904, Housings_SSOP:MSOP-8-1EP_3x3mm_Pitch0.65mm, symbol DS3904
- added W4: Y_REF, Wire_Pads:SolderWirePad_single_0-8mmDrill, symbol TEST_1P
- added W5: Z_REF, Wire_Pads:SolderWirePad_single_0-8mmDrill, symbol TEST_1P
- added W6: X_REF, Wire_Pads:SolderWirePad_single_0-8mmDrill, symbol TEST_1P
- added WXD7: XD0, Wire_Pads:SolderWirePad_single_0-8mmDrill, symbol TEST_1P
- added WXD8: XD1, Wire_Pads:SolderWirePad_single_0-8mmDrill, symbol TEST_1P
- added WYD1: YD0, Wire_Pads:SolderWirePad_single_0-8mmDrill, symbol TEST_1P
- added WYD2: YD1, Wire_Pads:SolderWirePad_single_0-8mmDrill, symbol TEST_1P
- added WZd0: ZD0, Wire_Pads:SolderWirePad_single_0-8mmDrill, symbol TEST_1P
- added WzD1: ZD1, Wire_Pads:SolderWirePad_single_0-8mmDrill, symbol TEST_1P
- P27: renamed from P205; value Y -> Y-MOT; footprint (none) -> Sockets_MOLEX_KK-System:Socket_MOLEX-KK-RM2-54mm_Lock_4pin_straight
- P28: renamed from P206; value Z -> Z-MOT1; footprint (none) -> Sockets_MOLEX_KK-System:Socket_MOLEX-KK-RM2-54mm_Lock_4pin_straight
- P29: renamed from P204; value X -> X-MOT; footprint (none) -> Sockets_MOLEX_KK-System:Socket_MOLEX-KK-RM2-54mm_Lock_4pin_straight
Connections:
- net labels added: +5V, GND-II_RevF_Date23Aug2012, SCL, SDA, X_TRIM, Y_TRIM, Z_TRIM, gnd, y-1B, y-2A, y-2B
- net labels removed: Y-1B, Y-2A, Y-2B
- wire segments 93 -> 258
- no-connect marks 0 -> 12
Other:
- note added: "X AXIS"
- note added: "Y AXIS"
- note added: "Z AXIS"
- moved on the sheet: P27, P28, P29
