File: RAMPS-FD/steppers2.sch (KiCad schematic (older format))
At the start: 15 parts, among them P207 CONN_3X2, P208 CONN_3X2, P209 CONN_3X2, P210 E2, P212 E1, P217 E0, U204 E2, U205 E1, U206 E0

Commit message: ramps-FD variant
Parts:
- removed C204, C205, C206: 100u 35V, symbol CP1
- removed P207, P208, P209: CONN_3X2, symbol CONN_3X2
- removed P210: E2, symbol CONN_4
- removed P212: E1, symbol CONN_4
- removed P217: E0, symbol CONN_4
- removed R207, R208, R210: 100k, symbol R
- removed U204: E2, symbol POLOLU
- removed U205: E1, symbol POLOLU
- removed U206: E0, symbol POLOLU
- added C10, C26, C8: 470n/10v, Capacitors_SMD:C_0805, symbol C
- added C11, C13, C28: 4u7/10v, Capacitors_SMD:C_0805, symbol C
- added C12, C15, C29: 100u/35v, Capacitors_SMD:c_elec_6.3x7.7, symbol CP1_Small
- added C14, C16, C30: 100n50v, Capacitors_SMD:C_0805, symbol C
- added C17, C19, C22, C24, C25, C31, C34, C7, C9: 100n/50v, Capacitors_SMD:C_0805, symbol C
- added C18, C20, C32: 22n/50v, Capacitors_SMD:C_0805, symbol C
- added C21, C23, C33: 1u/50v, Capacitors_SMD:C_0805, symbol C
- added C27: 0.1u, Capacitors_SMD:C_0805, symbol C_Small
- added P1: E1_SPRD_En, Pin_Headers:Pin_Header_Straight_1x02, symbol CONN_01X02
- added P10: E2-MOT, Sockets_MOLEX_KK-System:Socket_MOLEX-KK-RM2-54mm_Lock_4pin_straight, symbol CONN_4
- added P11: E0-MOT, Sockets_MOLEX_KK-System:Socket_MOLEX-KK-RM2-54mm_Lock_4pin_straight, symbol CONN_4
- added P32: E2_SPRD_En, Pin_Headers:Pin_Header_Straight_1x02, symbol CONN_01X02
- added P33: E0_SPRD_En, Pin_Headers:Pin_Header_Straight_1x02, symbol CONN_01X02
- added P9: E1-MOT, Sockets_MOLEX_KK-System:Socket_MOLEX-KK-RM2-54mm_Lock_4pin_straight, symbol CONN_4
- added R10, R11, R15, R16, R8, R9: 0r11, Resistors_SMD:R_0805, symbol R
- added R12, R6, R7: 2r2, Resistors_SMD:R_0805, symbol R
- added R13, R14: 4k7, Resistors_SMD:R_0805, symbol R
- added U5, U6, U8: TMC2130, Housings_DFN_QFN:QFN-36-1EP_5x6mm_Pitch0.5mm, symbol TMC2130-RESCUE-RAMPS-FD
- added U7: DS3904, Housings_SSOP:MSOP-8-1EP_3x3mm_Pitch0.65mm, symbol DS3904
- added W1: E1_REF, Wire_Pads:SolderWirePad_single_0-8mmDrill, symbol TEST_1P
- added W2: E2_REF, Wire_Pads:SolderWirePad_single_0-8mmDrill, symbol TEST_1P
- added W3: E0_REF, Wire_Pads:SolderWirePad_single_0-8mmDrill, symbol TEST_1P
- added WXD1: E1D0, Wire_Pads:SolderWirePad_single_0-8mmDrill, symbol TEST_1P
- added WXD2: E1D1, Wire_Pads:SolderWirePad_single_0-8mmDrill, symbol TEST_1P
- added WXD3: E2D0, Wire_Pads:SolderWirePad_single_0-8mmDrill, symbol TEST_1P
- added WXD4: E2D1, Wire_Pads:SolderWirePad_single_0-8mmDrill, symbol TEST_1P
- added WXD5: E0D0, Wire_Pads:SolderWirePad_single_0-8mmDrill, symbol TEST_1P
- added WXD6: E0D1, Wire_Pads:SolderWirePad_single_0-8mmDrill, symbol TEST_1P
Connections:
- net labels added: +5V, E0_TRIM, E1_TRIM, E2_TRIM, GND-II_RevF_Date23Aug2012, SCL, SDA, gnd
- wire segments 94 -> 253
- no-connect marks 0 -> 12
Other:
- note added: "E0 STEPPER"
- note added: "E1 STEPPER"
- note added: "E2 STEPPER"
