File: RAMPS-FD/thermistor_inputs.sch (KiCad schematic (older format))
At the start: 30 parts, among them P301 CONN_4X2, U1001 TL431_SOT23_RMC

Commit message: ramps-FD variant
Parts:
- C37: renamed from C504; footprint (none) -> Capacitors_SMD:C_0805; symbol C -> C-RESCUE-RAMPS-FD
- C38: renamed from C505; footprint (none) -> Capacitors_SMD:C_0805; symbol C -> C-RESCUE-RAMPS-FD
- C39: renamed from C503; footprint (none) -> Capacitors_SMD:C_0805; symbol C -> C-RESCUE-RAMPS-FD
- C40: renamed from C502; footprint (none) -> Capacitors_SMD:C_0805; symbol C -> C-RESCUE-RAMPS-FD
- C41: renamed from C301; footprint (none) -> Capacitors_SMD:C_0805; symbol C -> C-RESCUE-RAMPS-FD
- C42: renamed from C302; footprint (none) -> Capacitors_SMD:C_0805; symbol C -> C-RESCUE-RAMPS-FD
- C43: renamed from C303; footprint (none) -> Capacitors_SMD:C_0805; symbol C -> C-RESCUE-RAMPS-FD
- C44: renamed from C501; footprint (none) -> Capacitors_SMD:C_0805; symbol C -> C-RESCUE-RAMPS-FD
- C45: renamed from C1001; footprint ~ -> Capacitors_SMD:c_elec_4x5.3; symbol CP1 -> CP1-RESCUE-RAMPS-FD
- D17: renamed from D1003; footprint ~ -> Diodes_SMD:SOD-323; symbol DIODE -> DIODE-RESCUE-RAMPS-FD
- D18: renamed from D1004; footprint ~ -> Diodes_SMD:SOD-323; symbol DIODE -> DIODE-RESCUE-RAMPS-FD
- D19: renamed from D1005; footprint ~ -> Diodes_SMD:SOD-323; symbol DIODE -> DIODE-RESCUE-RAMPS-FD
- D20: renamed from D1006; footprint ~ -> Diodes_SMD:SOD-323; symbol DIODE -> DIODE-RESCUE-RAMPS-FD
- D21: renamed from D1001; footprint ~ -> Diodes_SMD:SOD-323; symbol DIODE -> DIODE-RESCUE-RAMPS-FD
- D22: renamed from D1002; footprint ~ -> Diodes_SMD:SOD-323; symbol DIODE -> DIODE-RESCUE-RAMPS-FD
- D23: renamed from D1007; footprint ~ -> Diodes_SMD:SOD-323; symbol DIODE -> DIODE-RESCUE-RAMPS-FD
- D24: renamed from D1008; footprint ~ -> Diodes_SMD:SOD-323; symbol DIODE -> DIODE-RESCUE-RAMPS-FD
- P26: renamed from P301; footprint (none) -> Pin_Headers:Pin_Header_Straight_2x04
- R33: renamed from R301; footprint (none) -> Resistors_SMD:R_0805; symbol R -> R-RESCUE-RAMPS-FD
- R34: renamed from R302; footprint (none) -> Resistors_SMD:R_0805; symbol R -> R-RESCUE-RAMPS-FD
- R35: renamed from R303; footprint (none) -> Resistors_SMD:R_0805; symbol R -> R-RESCUE-RAMPS-FD
- R36: renamed from R501; footprint (none) -> Resistors_SMD:R_0805; symbol R -> R-RESCUE-RAMPS-FD
- R37: renamed from R502; value 4k7 -> 1k; footprint (none) -> Resistors_SMD:R_0805; symbol R -> R-RESCUE-RAMPS-FD
- R38: renamed from R504; value 4k7 -> 1K; footprint (none) -> Resistors_SMD:R_0805; symbol R -> R-RESCUE-RAMPS-FD
- R39: renamed from R503; value 4k7 -> 1k; footprint (none) -> Resistors_SMD:R_0805; symbol R -> R-RESCUE-RAMPS-FD
- R40: renamed from R505; value 4k7 -> 1k; footprint (none) -> Resistors_SMD:R_0805; symbol R -> R-RESCUE-RAMPS-FD
- R41: renamed from R1002; value 6k8 -> 10k; footprint ~ -> Resistors_SMD:R_0805; symbol R -> R-RESCUE-RAMPS-FD
- R42: renamed from R1003; value 1k8 -> 1k5; footprint ~ -> Resistors_SMD:R_0805; symbol R -> R-RESCUE-RAMPS-FD
- R43: renamed from R1004; footprint ~ -> Resistors_SMD:R_0805; symbol R -> R-RESCUE-RAMPS-FD
- U12: renamed from U1001; footprint SOT23 -> TO_SOT_Packages_SMD:SOT-23
Connections:
- net labels added: AREF
- net labels removed: +V_LOGIC
- wire segments 76 -> 80
Other:
- note added: "From \nthermistor"
- note added: "Limit at 3.1V"
- note removed: "From \nthermistors"
- note removed: "Limit at about 3.1V"
